Commit message: addition of isaac sim support 	modified:   rover_description/CMakeLists.txt 	new file:   rover_description/config/ros2_control.yaml 	new file:   rover_description/launch/rsp.launch.py 	new file:   rover_description/ros2_control/ros2_control.xacro 	deleted:    rover_description/urdf/meshes/Assembly 1.stl 	new file:   rover_description/urdf/meshes/rover_base.stl 	new file:   rover_description/urdf/robot.urdf 	modified:   rover_description/urdf/robot.urdf.xacro 	modified:   rover_description/urdf/robot.xacro 	new file:   rover_description/urdf/robot/configuration/robot_base.usd 	new file:   rover_description/urdf/robot/configuration/robot_physics.usd 	new file:   rover_description/urdf/robot/configuration/robot_robot.usd 	new file:   rover_description/urdf/robot/configuration/robot_sensor.usd 	new file:   rover_description/urdf/robot/robot.usd

File: rover_description/urdf/robot.urdf.xacro (robot description, xacro)
@@ -2,3 +2,5 @@
 <robot xmlns:xacro="http://www.ros.org/wiki/xacro"  name="robot">
     <xacro:include filename="robot.xacro" />
+    <xacro:include filename="$(find rover_description)/ros2_control/ros2_control.xacro"/>
+    <xacro:rover_ros2_control name="RoverSystem"/>
 </robot>

File: rover_description/urdf/robot.xacro (robot description, xacro)
@@ -1,27 +1,48 @@
 <?xml version="1.0"?>
-<robot xmlns:xacro="http://www.ros.org/wiki/xacro" >
-    <xacro:include filename="inertial_macros.xacro"/>
-    <xacro:property name="wheel_radius" value="0.033"/>
+<robot xmlns:xacro="http://www.ros.org/wiki/xacro">
+    <xacro:property name="black" value="0 0 0 1"/>
+    <xacro:property name="blue" value="0 0 1 1"/>
+    <xacro:property name="grey" value="0.5 0.5 0.5 1"/>
+    <xacro:property name="wheel_radius" value="0.034"/>
     <xacro:property name="wheel_thickness" value="0.026"/>
     <xacro:property name="wheel_mass" value="0.05"/>
-    <xacro:property name="wheel_offset_x" value="0.226"/>
-    <xacro:property name="wheel_offset_y" value="0.1485"/>
-    <xacro:property name="wheel_offset_z" value="0.01"/>
+    <xacro:property name="front_wheel_offset_x" value="0.085"/>
+    <xacro:property name="rear_wheel_offset_x" value="0.085"/>
+    <xacro:property name="front_wheel_offset_y" value="0.038782"/>
+    <xacro:property name="rear_wheel_offset_y" value="0.070718"/>
+    <xacro:property name="wheel_offset_z" value="0.018845"/>
     <xacro:property name="base_mass" value="2.0"/>
-    <link name="base_link">
-    </link>
+    <link name="base_link"/>
     <link name="body_link">
         <visual>
+            <origin xyz="0 0 0" rpy="${pi/2} 0 0"/>
+            <material name="grey">
+                 <color rgba="${grey}"/>
+            </material>
+            <geometry>
+                <mesh
+                    filename="package://rover_description/urdf/meshes/rover_base.stl"
+                    scale="0.001 0.001 0.001"/>
+            </geometry>
+        </visual>
+        <collision>
+            <origin xyz="0 0 0" rpy="${pi/2} 0 0"/>
+            <geometry>
+                <mesh
+                    filename="package://rover_description/urdf/meshes/rover_base.stl"
+                    scale="0.001 0.001 0.001"/>
+            </geometry>
+        </collision>
+        <inertial>
             <origin xyz="0 0 0" rpy="0 0 0"/>
-            <geometry>
-                <mesh filename="meshes/Assembly.stl" scale="1.0"/>
-            </geometry>
-        </visual>
-        <collision>
-            <origin xyz="0 0 0" rpy="0 0 0"/>
-            <geometry>
-                <mesh filename="meshes/Assembly.stl" scale="1.0"/>
-            </geometry>
-        </collision>
+            <mass value="${base_mass}"/>
+            <inertia
+                ixx="0.1"
+                ixy="0.0"
+                ixz="0.0"
+                iyy="0.1"
+                iyz="0.0"
+                izz="0.1"/>
+        </inertial>
     </link>
     <joint name="body_joint" type="fixed">
@@ -29,5 +50,167 @@
         <child link="body_link"/>
         <origin xyz="0 0 0" rpy="0 0 0"/>
-        <axis xyz="0 0 0"/>
+    </joint>
+    <link name="back_left_wheel_link">
+        <visual>
+            <origin xyz="0 0 0" rpy="${pi/2} 0 ${pi/2}"/>
+            <material name="back">
+                 <color rgba="${black}"/>
+            </material>
+            <geometry>
+                <cylinder
+                    radius="${wheel_radius}"
+                    length="${wheel_thickness}"/>
+            </geometry>
+        </visual>
+        <collision>
+            <origin xyz="0 0 0" rpy="${pi/2} 0 ${pi/2}"/>
+            <geometry>
+                <cylinder
+                    radius="${wheel_radius}"
+                    length="${wheel_thickness}"/>
+            </geometry>
+        </collision>
+        <inertial>
+            <origin xyz="0 0 0" rpy="${pi/2} 0 ${pi/2}"/>
+            <mass value="${wheel_mass}"/>
+            <inertia
+                ixx="0.0001"
+                ixy="0.0"
+                ixz="0.0"
+                iyy="0.0001"
+                iyz="0.0"
+                izz="0.0001"/>
+        </inertial>
+    </link>
+    <joint name="back_left_wheel_joint" type="continuous">
+        <parent link="body_link"/>
+        <child link="back_left_wheel_link"/>
+        <origin
+            xyz="${-rear_wheel_offset_x} ${-rear_wheel_offset_y} ${wheel_offset_z}"
+            rpy="0 0 ${pi}"/>
+        <axis xyz="1 0 0"/>
+    </joint>
+    <!-- ================= BACK RIGHT WHEEL ================= -->
+    <link name="back_right_wheel_link">
+        <visual>
+            <origin xyz="0 0 0" rpy="${pi/2} 0 ${pi/2}"/>
+            <material name="back">
+                 <color rgba="${black}"/>
+            </material>
+            <geometry>
+                <cylinder
+                    radius="${wheel_radius}"
+                    length="${wheel_thickness}"/>
+            </geometry>
+        </visual>
+        <collision>
+            <origin xyz="0 0 0" rpy="${pi/2} 0 ${pi/2}"/>
+            <geometry>
+                <cylinder
+                    radius="${wheel_radius}"
+                    length="${wheel_thickness}"/>
+            </geometry>
+        </collision>
+        <inertial>
+            <origin xyz="0 0 0" rpy="${pi/2} 0 ${pi/2}"/>
+            <mass value="${wheel_mass}"/>
+            <inertia
+                ixx="0.0001"
+                ixy="0.0"
+                ixz="0.0"
+                iyy="0.0001"
+                iyz="0.0"
+                izz="0.0001"/>
+        </inertial>
+    </link>
+    <joint name="back_right_wheel_joint" type="continuous">
+        <parent link="body_link"/>
+        <child link="back_right_wheel_link"/>
+        <origin
+            xyz="${rear_wheel_offset_x} ${-rear_wheel_offset_y} ${wheel_offset_z}"
+            rpy="0 0 0"/>
+        <axis xyz="1 0 0"/>
+    </joint>
+    <!-- ================= FRONT LEFT WHEEL ================= -->
+    <link name="front_left_wheel_link">
+        <visual>
+            <origin xyz="0 0 0" rpy="-${pi/2} 0 ${pi/2}"/>
+            <material name="back">
+                 <color rgba="${black}"/>
+            </material>
+            <geometry>
+                <cylinder
+                    radius="${wheel_radius}"
+                    length="${wheel_thickness}"/>
+            </geometry>
+        </visual>
+        <collision>
+            <origin xyz="0 0 0" rpy="${pi/2} 0 ${pi/2}"/>
+            <geometry>
+                <cylinder
+                    radius="${wheel_radius}"
+                    length="${wheel_thickness}"/>
+            </geometry>
+        </collision>
+        <inertial>
+            <origin xyz="0 0 0" rpy="${pi/2} 0 ${pi/2}"/>
+            <mass value="${wheel_mass}"/>
+            <inertia
+                ixx="0.0001"
+                ixy="0.0"
+                ixz="0.0"
+                iyy="0.0001"
+                iyz="0.0"
+                izz="0.0001"/>
+        </inertial>
+    </link>
+    <joint name="front_left_wheel_joint" type="continuous">
+        <parent link="body_link"/>
+        <child link="front_left_wheel_link"/>
+        <origin
+            xyz="${-front_wheel_offset_x} ${front_wheel_offset_y} ${wheel_offset_z}"
+            rpy="0 0 ${pi}"/>
+        <axis xyz="1 0 0"/>
+    </joint>
+    <!-- ================= FRONT RIGHT WHEEL ================= -->
+    <link name="front_right_wheel_link">
+        <visual>
+            <origin xyz="0 0 0" rpy="${pi/2} 0 ${pi/2}"/>
+            <material name="black">
+                 <color rgba="${black}"/>
+            </material>
+            <geometry>
+                <cylinder
+                    radius="${wheel_radius}"
+                    length="${wheel_thickness}"/>
+            </geometry>
+        </visual>
+        <collision>
+            <origin xyz="0 0 0" rpy="${pi/2} 0 ${pi/2}"/>
+            <geometry>
+                <cylinder
+                    radius="${wheel_radius}"
+                    length="${wheel_thickness}"/>
+            </geometry>
+        </collision>
+        <inertial>
+            <origin xyz="0 0 0" rpy="${pi/2} 0 ${pi/2}"/>
+            <mass value="${wheel_mass}"/>
+            <inertia
+                ixx="0.0001"
+                ixy="0.0"
+                ixz="0.0"
+                iyy="0.0001"
+                iyz="0.0"
+                izz="0.0001"/>
+        </inertial>
+    </link>
+    <joint name="front_right_wheel_joint" type="continuous">
+        <parent link="body_link"/>
+        <child link="front_right_wheel_link"/>
+        <origin
+            xyz="${front_wheel_offset_x} ${front_wheel_offset_y} ${wheel_offset_z}"
+            rpy="0 0 0"/>
+        <axis xyz="1 0 0"/>
     </joint>
 </robot>
